Commit message: Add files via upload

File: src/arm_gripper_moveit_config/config/ARM.ros2_control.xacro (robot description, xacro)
@@ -6,5 +6,5 @@
             <hardware>
                 <!-- By default, set up controllers for simulation. This won't work on real hardware -->
-                <plugin>gazebo_ros2_control/GenericSystem</plugin>
+                <plugin>gazebo_ros2_control/GazeboSystem</plugin>
             </hardware>
             <joint name="revolute_1">
@@ -26,4 +26,11 @@
                 <state_interface name="position">
                   <param name="initial_value">${initial_positions['revolute_9']}</param>
+                </state_interface>
+                <state_interface name="velocity"/>
+            </joint>
+            <joint name="revolute_10">
+                <command_interface name="position"/>
+                <state_interface name="position">
+                  <param name="initial_value">${initial_positions['revolute_10']}</param>
                 </state_interface>
                 <state_interface name="velocity"/>

File: src/arm_gripper_moveit_config/config/ARM.urdf.xacro (robot description, xacro)
@@ -6,4 +6,4 @@
     <!-- Import control_xacro -->
     <xacro:include filename="ARM.ros2_control.xacro" />
-    <xacro:ARM_ros2_control name="FakeSystem" initial_positions_file="$(arg initial_positions_file)"/>
+    <!-- <xacro:ARM_ros2_control name="FakeSystem" initial_positions_file="$(arg initial_positions_file)"/> -->
 </robot>
